Commit message: Added 2 more volumetric spaces for the panda hand and the paper on the table

File: urdf/setup.urdf.xacro (robot description, xacro)
@@ -19,8 +19,38 @@
     </visual>
   </link>
-  <joint name="falcon_box_to_base" type="fixed">
+  <joint name="falcon_volume_to_base" type="fixed">
     <parent link="falcon_front"/>
     <child link="falcon_volume"/>
-    <origin xyz="0.12 0.0 0.0" rpy="${tau/2} ${-tau/4} ${tau/4}"/>
+    <origin xyz="0 0.0 0.12" rpy="${tau/2} ${-tau/4} ${tau/4}"/>
+  </joint>
+  <link name='panda_volume'>
+    <visual>
+        <geometry>
+            <box size="0.1 0.1 0.1"/>
+        </geometry>
+        <material name="blue_vol">
+            <color rgba="0.0 0.0 1.0 0.1"/>
+        </material>
+    </visual>
+  </link>
+  <joint name="panda_volume_to_hand" type="fixed">
+    <parent link="panda_hand_tcp"/>
+    <child link="panda_volume"/>
+    <origin xyz="0.0 0.0 0.0" rpy="${tau/2} 0 0"/>
+  </joint>
+  <link name='panda_table_volume'>
+    <visual>
+        <geometry>
+            <box size="0.1 0.1 0.1"/>
+        </geometry>
+        <material name="blue_vol">
+            <color rgba="0.0 0.0 1.0 0.1"/>
+        </material>
+    </visual>
+  </link>
+  <joint name="panda_volume_to_table" type="fixed">
+    <parent link="table_top"/>
+    <child link="panda_table_volume"/>
+    <origin xyz="0.0 0.0 0.05" rpy="0 0 0"/>
   </joint>
 </robot>

Commit message: absolute positon works

File: urdf/setup.urdf.xacro (robot description, xacro)
@@ -24,5 +24,5 @@
     <origin xyz="0 0.0 0.12" rpy="${tau/2} ${-tau/4} ${tau/4}"/>
   </joint>
-  <link name='panda_volume'>
+  <!-- <link name='panda_volume'>
     <visual>
         <geometry>
@@ -38,9 +38,9 @@
     <child link="panda_volume"/>
     <origin xyz="0.0 0.0 0.0" rpy="${tau/2} 0 0"/>
-  </joint>
+  </joint> -->
   <link name='panda_table_volume'>
     <visual>
         <geometry>
-            <box size="0.1 0.1 0.1"/>
+            <box size="0.5 0.5 0.5"/>
         </geometry>
         <material name="blue_vol">
@@ -52,5 +52,5 @@
     <parent link="table_top"/>
     <child link="panda_table_volume"/>
-    <origin xyz="0.0 0.0 0.05" rpy="0 0 0"/>
+    <origin xyz="0.0 0.2 0.29" rpy="0 0 0"/>
   </joint>
 </robot>

Commit message: Added the 2nd mode of control

File: urdf/setup.urdf.xacro (robot description, xacro)
@@ -22,5 +22,6 @@
     <parent link="falcon_front"/>
     <child link="falcon_volume"/>
-    <origin xyz="0 0.0 0.12" rpy="${tau/2} ${-tau/4} ${tau/4}"/>
+    <!-- <origin xyz="0 0.0 0.12" rpy="${tau/2} ${-tau/4} ${tau/4}"/> -->
+    <origin xyz="0 0.0 0.0" rpy="0 0 0"/>
   </joint>
   <!-- <link name='panda_volume'>
@@ -54,3 +55,18 @@
     <origin xyz="0.0 0.2 0.29" rpy="0 0 0"/>
   </joint>
+    <!-- <link name='falcon_volume_flipped'>
+    <visual>
+        <geometry>
+            <box size="0.1 0.1 0.1"/>
+        </geometry>
+        <material name="blue_vol">
+            <color rgba="0.0 0.0 1.0 0.1"/>
+        </material>
+    </visual>
+  </link>
+  <joint name="falcon_volume_flipped_to_base" type="fixed">
+    <parent link="falcon_front"/>
+    <child link="falcon_volume_flipped"/>
+    <origin xyz="0 0.0 0.12" rpy="${tau/2} ${-tau/2} ${tau/4}"/>
+  </joint> -->
 </robot>

Commit message: changed the mapper

File: urdf/setup.urdf.xacro (robot description, xacro)
@@ -12,5 +12,5 @@
     <visual>
         <geometry>
-            <box size="0.1 0.1 0.1"/>
+            <box size="0.08 0.1 0.1"/>
         </geometry>
         <material name="blue_vol">
@@ -22,6 +22,5 @@
     <parent link="falcon_front"/>
     <child link="falcon_volume"/>
-    <!-- <origin xyz="0 0.0 0.12" rpy="${tau/2} ${-tau/4} ${tau/4}"/> -->
-    <origin xyz="0 0.0 0.0" rpy="0 0 0"/>
+    <origin xyz="0 0.0 0.12" rpy="${tau/2} ${-tau/4} ${tau/4}"/>
   </joint>
   <!-- <link name='panda_volume'>
@@ -40,5 +39,5 @@
     <origin xyz="0.0 0.0 0.0" rpy="${tau/2} 0 0"/>
   </joint> -->
-  <link name='panda_table_volume'>
+  <!-- <link name='panda_table_volume'>
     <visual>
         <geometry>
@@ -54,5 +53,5 @@
     <child link="panda_table_volume"/>
     <origin xyz="0.0 0.2 0.29" rpy="0 0 0"/>
-  </joint>
+  </joint> -->
     <!-- <link name='falcon_volume_flipped'>
     <visual>

Commit message: fixed bugs

File: urdf/setup.urdf.xacro (robot description, xacro)
@@ -39,4 +39,10 @@
     <origin xyz="0.0 0.0 0.0" rpy="${tau/2} 0 0"/>
   </joint> -->
+  <link name='table_volume' />
+  <joint name="panda_volume_to_table_top" type="floating">
+    <parent link="table_top"/>
+    <child link="table_volume"/>
+    <origin xyz="0 0 0" rpy="0 0 0"/>
+  </joint>
   <!-- <link name='panda_table_volume'>
     <visual>

Commit message: added pen and made falcon in frame and rosbag record script

File: urdf/setup.urdf.xacro (robot description, xacro)
@@ -9,8 +9,8 @@
     <origin xyz="0 0.8 0.13" rpy="${tau/4} 0 ${tau/4}"/>
   </joint>
-  <link name='falcon_volume'>
+  <!-- <link name='falcon_volume'>
     <visual>
         <geometry>
-            <box size="0.08 0.1 0.1"/>
+            <box size="0.08 0.1 0.05"/>
         </geometry>
         <material name="blue_vol">
@@ -23,5 +23,5 @@
     <child link="falcon_volume"/>
     <origin xyz="0 0.0 0.12" rpy="${tau/2} ${-tau/4} ${tau/4}"/>
-  </joint>
+  </joint> -->
   <!-- <link name='panda_volume'>
     <visual>
@@ -45,4 +45,10 @@
     <origin xyz="0 0 0" rpy="0 0 0"/>
   </joint>
+  <!-- <link name='falcon_volume' />
+  <joint name="panda_volume_to_table_top" type="floating">
+    <parent link="table_top"/>
+    <child link="table_volume"/>
+    <origin xyz="0 0 0" rpy="${tau/2} ${-tau/4} ${tau/4}"/>
+  </joint> -->
   <!-- <link name='panda_table_volume'>
     <visual>
@@ -75,3 +81,25 @@
     <origin xyz="0 0.0 0.12" rpy="${tau/2} ${-tau/2} ${tau/4}"/>
   </joint> -->
+<link name="pen">
+  <visual>
+    <origin xyz="0 0 -0.0635" rpy="0 0 0"/>
+    <geometry>
+      <cylinder radius="0.01" length="0.127"/>
+    </geometry>
+    <material name="pen_rad">
+      <color rgba="0.0 1.0 0.0 0.5"/>
+    </material>
+  </visual>
+  <!-- <collision>
+    <origin xyz="0 0 -0.0635 " rpy="0 0 0"/>
+    <geometry>
+      <cylinder radius="0.01" length="0.127"/>
+    </geometry>
+  </collision> -->
+</link>
+<joint name="pen_joint" type="fixed">
+  <parent link="panda_hand_tcp"/>
+  <child link="pen"/>
+  <origin xyz="0 0 0.09" rpy="0 0 0"/>
+</joint>
 </robot>

Commit message: works

File: urdf/setup.urdf.xacro (robot description, xacro)
@@ -85,5 +85,5 @@
     <origin xyz="0 0 -0.0635" rpy="0 0 0"/>
     <geometry>
-      <cylinder radius="0.01" length="0.127"/>
+      <cylinder radius="0.01" length="0.12"/>
     </geometry>
     <material name="pen_rad">
@@ -101,5 +101,5 @@
   <parent link="panda_hand_tcp"/>
   <child link="pen"/>
-  <origin xyz="0 0 0.09" rpy="0 0 0"/>
+  <origin xyz="0 0 0.0935" rpy="0 0 0"/>
 </joint>
 </robot>

Commit message: finalising the 1.0

File: urdf/setup.urdf.xacro (robot description, xacro)
@@ -85,5 +85,5 @@
     <origin xyz="0 0 -0.0635" rpy="0 0 0"/>
     <geometry>
-      <cylinder radius="0.01" length="0.12"/>
+      <cylinder radius="0.0083" length="0.129"/>
     </geometry>
     <material name="pen_rad">
@@ -101,5 +101,5 @@
   <parent link="panda_hand_tcp"/>
   <child link="pen"/>
-  <origin xyz="0 0 0.0935" rpy="0 0 0"/>
+  <origin xyz="0 0 0.097" rpy="0 0 0"/>
 </joint>
 </robot>
